Commit message: made code easy to read

File: urdf/ur5_7thaxis.urdf (robot description, URDF)
Before this commit: robot ur5e, 18 links, 17 joints
Links:
- link trees: geometry collision mesh filename=package://masters_project/meshes/ufo_trees_labelled/2.stl scale=.1 .1 .1; visual mesh filename=package://masters_project/meshes/ufo_trees_labelled/2.stl scale=.1 .1 .1

Commit message: coding done and PID working

File: urdf/ur5_7thaxis.urdf (robot description, URDF)
Before this commit: robot ur5e, 18 links, 17 joints
Links:
- link trees: geometry collision mesh filename=package://masters_project/meshes/ufo_trees_labelled/2.stl scale=.1 .1 .1; visual mesh filename=package://masters_project/meshes/ufo_trees_labelled/0.stl scale=.1 .1 .1

Commit message: flownet with Cindy's curve fitting

File: urdf/ur5_7thaxis.urdf (robot description, URDF)
Before this commit: robot ur5e, 18 links, 17 joints
Links:
- removed link trees
- added link tree_0; collision mesh filename=package://masters_project/meshes/ufo_trees_labelled/0.stl scale=.1 .1 .1; visual mesh filename=package://masters_project/meshes/ufo_trees_labelled/0.stl scale=.1 .1 .1
- added link tree_1; collision mesh filename=package://masters_project/meshes/ufo_trees_labelled/1.stl scale=.1 .1 .1; visual mesh filename=package://masters_project/meshes/ufo_trees_labelled/1.stl scale=.1 .1 .1
Joints:
- removed joint world_tree_fixed_joint
- added joint world_tree0_fixed_joint: type fixed, parent world, child tree_0, origin xyz=0 0 0 rpy=0.0 0.0 0.0
- added joint world_tree1_fixed_joint: type fixed, parent world, child tree_1, origin xyz=0 0 0 rpy=0.0 0.0 0.0

Commit message: added trees

File: urdf/ur5_7thaxis.urdf (robot description, URDF)
Before this commit: robot ur5e, 19 links, 18 joints
Links:
- removed link tree_0
- removed link tree_1
Joints:
- removed joint world_tree0_fixed_joint
- removed joint world_tree1_fixed_joint

Commit message: major refactor of the mask/curve logic to return all masks, adds logic in controller/image processor for using priors and avoiding large jumps

File: urdf/ur5_7thaxis.urdf (robot description, URDF)
Before this commit: robot ur5e, 17 links, 16 joints
Links:
- removed link cutpoint
- removed link cutter
- removed link endpoint
Joints:
- removed joint cutpoint
- removed joint cutter
- removed joint endpoint
